File: Traeger rev 2.3.0.kicad_pro.kicad_pcb (KiCad board)
At the start: 2 copper layers, 129.9 x 63.6 mm, 45 parts, among them J1 MAX6675, J10 Buttons, J2 Time of Flight Sensor, J3 MAX31865-RTD, J5 Rotary Encoder, J6 ADS1115 0x49, J7 Temp Sensors, J8 Temp Sensors, J9 Conn_01x06_Socket, K1 Fan Relay, K3 Auger 1 Relay, K6 Igniter 1 Relay, Q1 BC547, Q2 BC547, Q6 BC547, U1 ESP32-S3-DevKitC

Commit message: Update KiCad schematic and PCB for hardware changes
- ADS1115 VCC moved from 5V to 3.3V rail
- Pull-down resistors R_A0/R_A1 changed from 150kΩ to 1kΩ

Co-Authored-By: Claude Sonnet 4.6 <noreply@anthropic.com>
Parts:
- K1: value Fan Relay -> Fan SSR - OMRON G3MC-202PL
- K3: value Auger 1 Relay -> Auger SSR - OMRON G3MC-202PL
- K6: value Igniter 1 Relay -> Igniter SSR - OMRON G3MC-202PL
- R4, R5: value 150k -> 1k
Connections:
- J5 pad 2: VCC -> 3V3
- J6 pad 1: VCC -> 3V3
- J6 pad 5: VCC -> 3V3
- J7 pad 2: VCC -> 3V3
- J7 pad 4: VCC -> 3V3
- J8 pad 2: VCC -> 3V3
- J8 pad 4: VCC -> 3V3
Routing:
- net 3V3: track 69.8 -> 186.3 mm, vias 0 -> 2
- net VCC: track 292.0 -> 237.1 mm
- net SMOKE SW: track 67.5 -> 64.8 mm, vias 1 -> 0
